File: Temp sensor.kicad_sch (KiCad schematic)
At the start: 1 part, among them U1 ProS3

Commit message: A
Parts:
- added R1: 4700Ω, symbol Device:R
- added Temp1, Temp2: DS18B20, Package_TO_SOT_THT:TO-92_Inline, symbol Sensor_Temperature:DS18B20
Connections:
- net at U1.2 (GND): now also Temp1.1 (GND), Temp2.1 (GND)
- net at U1.4 (3V3): now also R1.1, Temp1.3 (V_{DD}), Temp2.3 (V_{DD})
- net at U1.5 (IO1): now also R1.2, Temp1.2 (DQ), Temp2.2 (DQ)
Changed lines of the file:
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@@
 (kicad_sch (version 20230121) (generator eeschema)
   (paper "A4")
-  (wire (pts (xy 107.95 72.39) (xy 137.16 72.39))
-    (stroke (width 0) (type default))
-  )
-  (wire (pts (xy 107.95 69.85) (xy 137.16 69.85))
-    (stroke (width 0) (type default))
-  )
-  (wire (pts (xy 107.95 64.77) (xy 137.16 64.77))
-    (stroke (width 0) (type default))
+  (junction (at 137.16 69.85) (diameter 0) (color 0 0 0 0)
+  )
+  (junction (at 119.38 69.85) (diameter 0) (color 0 0 0 0)
+  )
+  (junction (at 147.32 64.77) (diameter 0) (color 0 0 0 0)
+  )
+  (junction (at 119.38 80.01) (diameter 0) (color 0 0 0 0)
+  )
+  (junction (at 142.24 80.01) (diameter 0) (color 0 0 0 0)
+  )
+  (wire (pts (xy 107.95 64.77) (xy 147.32 64.77))
+    (stroke (width 0) (type default))
+  )
+  (wire (pts (xy 114.3 72.39) (xy 114.3 80.01))
+    (stroke (width 0) (type default))
+  )
+  (wire (pts (xy 119.38 78.74) (xy 119.38 80.01))
+    (stroke (width 0) (type default))
+  )
+  (wire (pts (xy 107.95 72.39) (xy 114.3 72.39))
+    (stroke (width 0) (type default))
+  )
+  (wire (pts (xy 147.32 64.77) (xy 147.32 87.63))
+    (stroke (width 0) (type default))
+  )
+  (wire (pts (xy 160.02 63.5) (xy 160.02 69.85))
+    (stroke (width 0) (type default))
+  )
+  (wire (pts (xy 142.24 69.85) (xy 142.24 80.01))
+    (stroke (width 0) (type default))
+  )
+  (wire (pts (xy 167.64 99.06) (xy 167.64 87.63))
+    (stroke (width 0) (type default))
+  )
+  (wire (pts (xy 152.4 55.88) (xy 147.32 55.88))
+    (stroke (width 0) (type default))
+  )
+  (wire (pts (xy 167.64 43.18) (xy 167.64 55.88))
+    (stroke (width 0) (type default))
+  )
+  (wire (pts (xy 147.32 87.63) (xy 152.4 87.63))
+    (stroke (width 0) (type default))
+  )
+  (wire (pts (xy 107.95 69.85) (xy 119.38 69.85))
+    (stroke (width 0) (type default))
+  )
+  (wire (pts (xy 114.3 80.01) (xy 119.38 80.01))
+    (stroke (width 0) (type default))
+  )
+  (wire (pts (xy 137.16 43.18) (xy 137.16 69.85))
+    (stroke (width 0) (type default))
+  )
+  (wire (pts (xy 160.02 69.85) (xy 142.24 69.85))
+    (stroke (width 0) (type default))
+  )
+  (wire (pts (xy 119.38 69.85) (xy 119.38 71.12))
+    (stroke (width 0) (type default))
+  )
+  (wire (pts (xy 142.24 95.25) (xy 160.02 95.25))
+    (stroke (width 0) (type default))
+  )
+  (wire (pts (xy 147.32 55.88) (xy 147.32 64.77))
+    (stroke (width 0) (type default))
+  )
+  (wire (pts (xy 119.38 69.85) (xy 137.16 69.85))
+    (stroke (width 0) (type default))
+  )
+  (wire (pts (xy 137.16 69.85) (xy 137.16 99.06))
+    (stroke (width 0) (type default))
+  )
+  (wire (pts (xy 142.24 80.01) (xy 142.24 95.25))
+    (stroke (width 0) (type default))
+  )
+  (wire (pts (xy 137.16 99.06) (xy 167.64 99.06))
+    (stroke (width 0) (type default))
+  )
+  (wire (pts (xy 137.16 43.18) (xy 167.64 43.18))
+    (stroke (width 0) (type default))
+  )
+  (wire (pts (xy 119.38 80.01) (xy 142.24 80.01))
+    (stroke (width 0) (type default))
+  )
+  (symbol (lib_id "Sensor_Temperature:DS18B20") (at 160.02 55.88 270) (unit 1)
+    (in_bom yes) (on_board yes) (dnp no) (fields_autoplaced)
+    (property "Reference" "Temp1" (at 160.02 45.72 90)
+      (effects (font (size 1.27 1.27)))
+    )
+    (property "Value" "DS18B20" (at 160.02 48.26 90)
+      (effects (font (size 1.27 1.27)))
+    )
+    (property "Footprint" "Package_TO_SOT_THT:TO-92_Inline" (at 153.67 30.48 0)
+      (effects (font (size 1.27 1.27)) hide)
+    )
+    (property "Datasheet" "http://datasheets.maximintegrated.com/en/ds/DS18B20.pdf" (at 166.37 52.07 0)
+      (effects (font (size 1.27 1.27)) hide)
+    )
+    (pin "1")
+    (pin "3")
+    (pin "2")
+    (instances
+      (project "Temp sensor"
+        (path "/8180f0fc-d351-47ff-bffa-772ac3a577c5"
+          (reference "Temp1") (unit 1)
+        )
+      )
+    )
+  )
+  (symbol (lib_id "Sensor_Temperature:DS18B20") (at 160.02 87.63 270) (unit 1)
+    (in_bom yes) (on_board yes) (dnp no) (fields_autoplaced)
+    (property "Reference" "Temp2" (at 160.02 77.47 90)
+      (effects (font (size 1.27 1.27)))
+    )
+    (property "Value" "DS18B20" (at 160.02 80.01 90)
+      (effects (font (size 1.27 1.27)))
+    )
+    (property "Footprint" "Package_TO_SOT_THT:TO-92_Inline" (at 153.67 62.23 0)
+      (effects (font (size 1.27 1.27)) hide)
+    )
+    (property "Datasheet" "http://datasheets.maximintegrated.com/en/ds/DS18B20.pdf" (at 166.37 83.82 0)
+      (effects (font (size 1.27 1.27)) hide)
+    )
+    (pin "2")
+    (pin "1")
+    (pin "3")
+    (instances
+      (project "Temp sensor"
+        (path "/8180f0fc-d351-47ff-bffa-772ac3a577c5"
+          (reference "Temp2") (unit 1)
+        )
+      )
+    )
   )
   (symbol (lib_id "ProS3:ProS3") (at 93.98 82.55 0) (unit 1)
@@
     (pin "9")
     (instances
-      (project "Rover"
+      (project "Temp sensor"
         (path "/8180f0fc-d351-47ff-bffa-772ac3a577c5"
           (reference "U1") (unit 1)
         )
       )
+    )
+  )
+  (symbol (lib_id "Device:R") (at 119.38 74.93 0) (unit 1)
+    (in_bom yes) (on_board yes) (dnp no) (fields_autoplaced)
+    (property "Reference" "R1" (at 121.92 73.66 0)
+      (effects (font (size 1.27 1.27)) (justify left))
+    )
+    (property "Value" "4700Ω" (at 121.92 76.2 0)
+      (effects (font (size 1.27 1.27)) (justify left))
+    )
+    (property "Footprint" "" (at 117.602 74.93 90)
+      (effects (font (size 1.27 1.27)) hide)
+    )
+    (property "Datasheet" "~" (at 119.38 74.93 0)
+      (effects (font (size 1.27 1.27)) hide)
+    )
+    (pin "1")
+    (pin "2")
+    (instances
+      (project "Temp sensor"
+        (path "/8180f0fc-d351-47ff-bffa-772ac3a577c5"
+          (reference "R1") (unit 1)
+        )
+      )
